Commit message: feat: Add MID360 support

File: config/robot.urdf.xacro (robot description, xacro)
@@ -9,8 +9,8 @@
     <origin xyz="0 0 0" rpy="0 0 0" />
   </joint>
-  <link name="lidar_link"> </link>
+  <link name="livox_frame"> </link>
   <joint name="lidar_joint" type="fixed">
     <parent link="base_link" />
-    <child link="lidar_link" />
+    <child link="livox_frame" />
     <origin xyz="0 0 0" rpy="0 0 0" />
   </joint>
